Commit message: 1

File: source/robot_lab/data/Robots/roboparty/atom01_description/urdf/atom01.urdf (robot description, URDF)
Before this commit: robot atom01urdf, 24 links, 23 joints
Links:
- link base_link: mass 5.18128957 -> 5.38006123; geometry collision mesh filename=./meshes/base_link.STL; visual mesh filename=./meshes/base_link.STL
- link left_ankle_pitch_link: mass 0.08430000 -> 0.084; geometry visual mesh filename=./meshes/left_ankle_pitch_link.STL
- link left_ankle_roll_link: mass 0.25150733 -> 0.30640039 ; geometry collision mesh filename=./meshes/left_ankle_roll_link.STL; visual mesh filename=./meshes/left_ankle_roll_link.STL
- link left_arm_pitch_link: mass 0.46177377 -> 0.47178757; geometry collision cylinder length=0.05 radius=0.03; visual mesh filename=./meshes/left_arm_pitch_link.STL
- link left_arm_roll_link: mass 0.07920766 -> 0.09168685; geometry collision cylinder length=0.10 radius=0.03; visual mesh filename=./meshes/left_arm_roll_link.STL
- link left_arm_yaw_link: mass 1.16138345 -> 1.15324429; geometry collision cylinder length=0.05 radius=0.03; visual mesh filename=./meshes/left_arm_yaw_link.STL
- link left_elbow_pitch_link: mass 0.07920766 -> 0.09168685; geometry collision cylinder length=0.10 radius=0.03; visual mesh filename=./meshes/left_elbow_pitch_link.STL
- link left_elbow_yaw_link: mass 0.69960968 -> 0.68145673; geometry visual mesh filename=./meshes/left_elbow_yaw_link.STL
- link left_knee_link: mass  1.57203189 -> 1.79036871; geometry collision box name=right_knee_link size=0.08 0.08 0.22; visual mesh filename=./meshes/left_knee_link.STL
- link left_thigh_pitch_link: mass 2.40451173 -> 2.34600762; geometry collision box name=left_thigh_pitch_link size=0.08 0.1 0.22; visual mesh filename=./meshes/left_thigh_pitch_link.STL
- link left_thigh_roll_link: mass 1.66242030 -> 1.71632646; geometry visual mesh filename=./meshes/left_thigh_roll_link.STL
- link left_thigh_yaw_link: mass 1.65548536 -> 1.68866185; geometry visual mesh filename=./meshes/left_thigh_yaw_link.STL
- link right_ankle_pitch_link: mass 0.08430000 -> 0.084; geometry visual mesh filename=./meshes/right_ankle_pitch_link.STL
- link right_ankle_roll_link: mass 0.25150733 ->  0.30640039; geometry collision mesh filename=./meshes/right_ankle_roll_link.STL; visual mesh filename=./meshes/right_ankle_roll_link.STL
- link right_arm_pitch_link: mass 0.46177377 -> 0.47178757; geometry collision cylinder length=0.05 radius=0.03; visual mesh filename=./meshes/right_arm_pitch_link.STL
- link right_arm_roll_link: mass 0.07920766 -> 0.09168685; geometry collision cylinder length=0.10 radius=0.03; visual mesh filename=./meshes/right_arm_roll_link.STL
- link right_arm_yaw_link: mass 1.16138345 -> 1.15324429; geometry collision cylinder length=0.05 radius=0.03; visual mesh filename=./meshes/right_arm_yaw_link.STL
- link right_elbow_pitch_link: mass 0.07920766 -> 0.09168685; geometry collision cylinder length=0.10 radius=0.03; visual mesh filename=./meshes/right_elbow_pitch_link.STL
- link right_elbow_yaw_link: mass 0.69960968 -> 0.68145673; geometry visual mesh filename=./meshes/right_elbow_yaw_link.STL
- link right_knee_link: mass 1.57203189 -> 1.79036871; geometry collision box name=right_knee_link size=0.08 0.08 0.22; visual mesh filename=./meshes/right_knee_link.STL
- link right_thigh_pitch_link: mass 2.40451173 -> 2.34600762; geometry collision box name=right_thigh_pitch_link size=0.08 0.1 0.22; visual mesh filename=./meshes/right_thigh_pitch_link.STL
- link right_thigh_roll_link: mass  1.66242030 -> 1.71632646; geometry visual mesh filename=./meshes/right_thigh_roll_link.STL
- link right_thigh_yaw_link: mass 1.65548536 -> 1.68565743; geometry visual mesh filename=./meshes/right_thigh_yaw_link.STL
- link torso_link: mass 6.57129050 -> 7.70005232 ; geometry collision box name=torso_link size=0.16 0.16 0.22; visual mesh filename=./meshes/torso_link.STL
Joints:
- joint left_ankle_pitch_joint: origin xyz=0 -0.024814 -0.3 rpy=0 0 0 -> xyz=0 -0.02085 -0.3 rpy=0 0 0
- joint left_arm_pitch_joint: limit lower=-2.0 upper=2.0 effort=18 velocity=3.7692 -> lower=-1.57 upper=1.57 effort=18 velocity=3.7692; origin xyz=0 0.12175 0.20518 rpy=0 0 0 -> xyz=0 0.121749999999383 0.206175860782433 rpy=0 0 0
- joint left_arm_roll_joint: limit lower=-0.25 upper=2.25 effort=18 velocity=3.7692 -> lower=-0.25 upper=1 effort=18 velocity=3.7692; origin xyz=0.02 0.056 0 rpy=0 0 0 -> xyz=0.0200000000000018 0.056 0 rpy=0 0 0
- joint left_arm_yaw_joint: limit lower=-2.6 upper=2.6 effort=18 velocity=3.7692 -> lower=-1.57 upper=1.57 effort=18 velocity=3.7692; origin xyz=-0.02 0 -0.05 rpy=0 0 0 -> xyz=-0.0200000000000002 0 -0.049999999999998 rpy=0 0 0
- joint left_elbow_pitch_joint: limit lower=-1.0 upper=1.57 effort=18 velocity=3.7692 -> lower=-0.6 upper=1.57 effort=18 velocity=3.7692; origin xyz=0 0.02 -0.18875 rpy=0 0 0 -> xyz=0 0.0199999999999982 -0.188749999999997 rpy=0 0 0
- joint left_elbow_yaw_joint: origin xyz=0.05 -0.02 0 rpy=0 0 0 -> xyz=0.0499999999999968 -0.0199999999999994 0 rpy=0 0 0
- joint left_knee_joint: limit lower=0 upper=2.5 effort=80 velocity=10.47 -> lower=-0.2 upper=2.5 effort=80 velocity=10.47; origin xyz=0 3.0016E-05 -0.25 rpy=0 0 0 -> xyz=0 0 -0.25 rpy=0 0 0
- joint left_thigh_pitch_joint: limit lower=-2.5 upper=0.8 effort=80 velocity=10.47 -> lower=-1 upper=1 effort=80 velocity=10.47; origin xyz=0.057159 0.02485 -0.032997 rpy=0 0 0 -> xyz=0.060622 0.02085 -0.035 rpy=0 0 0
- joint left_thigh_roll_joint: limit lower=-0.2 upper=2 effort=80 velocity=10.47 -> lower=-0.2 upper=1 effort=80 velocity=10.47; origin xyz=-0.014479 0 -0.074779 rpy=0 0 0 -> xyz=-0.017693 0 -0.072346 rpy=0 0 0
- joint left_thigh_yaw_joint: origin xyz=-0.10111 0.072188 -0.0014904 rpy=0 0 0 -> xyz=-0.071093 0.0725 -0.051778 rpy=0 0 0
- joint right_ankle_pitch_joint: origin xyz=0 0.024886 -0.3 rpy=0 0 0 -> xyz=0 0.0208500000000073 -0.299999999999986 rpy=0 0 0
- joint right_arm_pitch_joint: limit lower=-2 upper=2 effort=18 velocity=3.7692 -> lower=-1.57 upper=1.57 effort=18 velocity=3.7692; origin xyz=0 -0.12175 0.20518 rpy=0 0 0 -> xyz=0 -0.121750000000346 0.206175860781721 rpy=0 0 0
- joint right_arm_roll_joint: limit lower=-2.25 upper=0.25 effort=18 velocity=3.7692 -> lower=-1 upper=0.25 effort=18 velocity=3.7692; origin xyz=0.02 -0.056 0 rpy=0 0 0 -> xyz=0.0200000000000407 -0.056 0 rpy=0 0 0
- joint right_arm_yaw_joint: limit lower=-2.6 upper=2.6 effort=18 velocity=3.7692 -> lower=-1.57 upper=1.57 effort=18 velocity=3.7692; origin xyz=-0.02 0 -0.05 rpy=0 0 0 -> xyz=-0.02 0 -0.0500000000000019 rpy=0 0 0
- joint right_elbow_pitch_joint: limit lower=-1.0 upper=1.57 effort=18 velocity=3.7692 -> lower=-0.6 upper=1.57 effort=18 velocity=3.7692; origin xyz=0 -0.02 -0.18875 rpy=0 0 0 -> xyz=0 -0.0200000000000019 -0.18875 rpy=0 0 0
- joint right_elbow_yaw_joint: origin xyz=0.05 0.02 0 rpy=0 0 0 -> xyz=0.0500000000000002 0.0200000000000004 0 rpy=0 0 0
- joint right_knee_joint: limit lower=0 upper=2.5 effort=80 velocity=10.47 -> lower=-0.2 upper=2.5 effort=80 velocity=10.47; origin xyz=0 3.0016E-05 -0.25 rpy=0 0 0 -> xyz=0 0 -0.250000000000016 rpy=0 0 0
- joint right_thigh_pitch_joint: limit lower=-2.5 upper=0.8 effort=80 velocity=10.47 -> lower=-1 upper=1 effort=80 velocity=10.47; origin xyz=0.057156 -0.02485 -0.033003 rpy=0 0 0 -> xyz=0.0619208163652291 -0.0208499999999942 -0.0357500000093095 rpy=0 0 0
- joint right_thigh_roll_joint: limit lower=-2 upper=0.2 effort=80 velocity=10.47 -> lower=-1 upper=0.2 effort=80 velocity=10.47; origin xyz=-0.011479 0 -0.069583 rpy=0 0 0 -> xyz=-0.0189924084475403 0 -0.0715958163677252 rpy=0 0 0
- joint right_thigh_yaw_joint: origin xyz=-0.10411 -0.072812 -0.0066865 rpy=0 0 0 -> xyz=-0.071093 -0.0725 -0.051778 rpy=0 0 0
- joint torso_joint: limit lower=-2.62 upper=2.62 effort=80 velocity=10.47 -> lower=-3.14 upper=3.14 effort=80 velocity=10.47; origin xyz=-0.058434 -0.00031196 0.11805 rpy=0 0 0 -> xyz=-0.0281649492242451 0 0.0672000000054882 rpy=0 0 0
